File: 12v_lamp.kicad_pcb (KiCad board)
At the start: 2 copper layers, 137.5 x 40 mm, 50 parts, among them J1 Barrel_Jack_Switch, Q1 DMG2302U, SW1 SW_SPST

Commit message: Add logo
Parts:
- added REF**: Logo_WM, Symbol:Logo_WM, B.Cu at (69.7, 58.0)
Other:
- board text added: "v0.0.0 01/24/21"
